File: CH569Board.kicad_sch (KiCad schematic)
At the start: 36 parts, among them CN1 BA42-80BT-1-NHB, J1 Conn_01x02_Male, J2 Conn_01x03_Male, U1 AMS1117-3.3, U3 W25Q32JVSSIQ, U4 CH569W, X1 O705030MEEA4SC

Commit message: add decoupling caps in serdes, layout improvements
Parts:
- added C21, C22: 100nF, Capacitor_SMD:C_0402_1005Metric, symbol jlcpcb-basic-mlcc-0402:100nF
- U2: value (none) -> AMS1117-1.2
Connections:
- net GX+: now also C21.2; no longer J1.1 (Pin_1)
- net GX-: now also C22.2; no longer J1.2 (Pin_2)
- new net: C22.1, J1.2 (Pin_2)
- new net: C21.1, J1.1 (Pin_1)
Other:
- moved on the sheet: J1
Changed lines of the file:
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@@
+    (stroke (width 0) (type default) (color 0 0 0 0))
+  )
+  (wire (pts (xy 77.978 177.292) (xy 72.644 177.292))
     (stroke (width 0) (type default) (color 0 0 0 0))
   )
@@
     (stroke (width 0) (type default) (color 0 0 0 0))
   )
-  (wire (pts (xy 101.092 148.336) (xy 93.98 148.336))
+  (wire (pts (xy 90.17 181.61) (xy 83.058 181.61))
     (stroke (width 0) (type default) (color 0 0 0 0))
   )
@@
     (stroke (width 0) (type default) (color 0 0 0 0))
   )
-  (wire (pts (xy 101.092 145.796) (xy 93.98 145.796))
+  (wire (pts (xy 90.17 177.292) (xy 83.058 177.292))
     (stroke (width 0) (type default) (color 0 0 0 0))
   )
@@
     (stroke (width 0) (type default) (color 0 0 0 0))
   )
+  (wire (pts (xy 72.644 177.292) (xy 72.644 178.308))
+    (stroke (width 0) (type default) (color 0 0 0 0))
+  )
   (wire (pts (xy 166.624 99.314) (xy 171.196 99.314))
     (stroke (width 0) (type default) (color 0 0 0 0))
@@
     (stroke (width 0) (type default) (color 0 0 0 0))
   )
+  (wire (pts (xy 72.644 181.61) (xy 72.644 180.848))
+    (stroke (width 0) (type default) (color 0 0 0 0))
+  )
   (wire (pts (xy 120.65 64.77) (xy 133.096 64.77))
     (stroke (width 0) (type default) (color 0 0 0 0))
@@
   )
   (wire (pts (xy 147.828 56.896) (xy 156.21 56.896))
+    (stroke (width 0) (type default) (color 0 0 0 0))
+  )
+  (wire (pts (xy 77.978 181.61) (xy 72.644 181.61))
     (stroke (width 0) (type default) (color 0 0 0 0))
   )
@@
     (effects (font (size 1.27 1.27)) (justify left bottom))
   )
-  (label "GX+" (at 96.266 145.796 0)
+  (label "GX+" (at 85.344 177.292 0)
     (effects (font (size 1.27 1.27)) (justify left bottom))
   )
@@
     (effects (font (size 1.27 1.27)) (justify left bottom))
   )
-  (label "GX-" (at 96.266 148.336 0)
+  (label "GX-" (at 85.344 181.61 0)
     (effects (font (size 1.27 1.27)) (justify left bottom))
   )
@@
     (pin "8")
   )
+  (symbol (lib_id "jlcpcb-basic-mlcc-0402:100nF") (at 80.518 181.61 90) (unit 1)
+    (in_bom yes) (on_board yes)
+    (property "Reference" "C22" (id 0) (at 80.518 185.166 90))
+    (property "Value" "100nF" (id 1) (at 80.518 187.706 90))
+    (property "Footprint" "Capacitor_SMD:C_0402_1005Metric" (id 2) (at 84.328 180.6448 0)
+      (effects (font (size 1.27 1.27)) hide)
+    )
+    (property "Datasheet" "https://datasheet.lcsc.com/szlcsc/Samsung-Electro-Mechanics-CL05B104KO5NNNC_C1525.pdf" (id 3) (at 80.518 181.61 90)
+      (effects (font (size 1.27 1.27)) hide)
+    )
+    (property "LCSC" "C1525" (id 4) (at 80.518 181.61 90)
+      (effects (font (size 1.27 1.27)) hide)
+    )
+    (pin "1")
+    (pin "2")
+  )
   (symbol (lib_id "Device:C_Small") (at 77.978 44.196 180) (unit 1)
     (in_bom yes) (on_board yes)
@@
     (pin "1")
   )
-  (symbol (lib_id "Connector:Conn_01x02_Male") (at 88.9 145.796 0) (unit 1)
-    (in_bom yes) (on_board yes)
-    (property "Reference" "J1" (id 0) (at 88.9 143.764 0))
-    (property "Value" "Conn_01x02_Male" (id 1) (at 93.726 150.876 0))
-    (property "Footprint" "Connector_PinHeader_1.00mm:PinHeader_1x02_P1.00mm_Vertical" (id 2) (at 88.9 145.796 0)
-      (effects (font (size 1.27 1.27)) hide)
-    )
-    (property "Datasheet" "~" (id 3) (at 88.9 145.796 0)
+  (symbol (lib_id "Connector:Conn_01x02_Male") (at 67.564 178.308 0) (unit 1)
+    (in_bom yes) (on_board yes)
+    (property "Reference" "J1" (id 0) (at 67.564 176.276 0))
+    (property "Value" "Conn_01x02_Male" (id 1) (at 72.39 183.388 0))
+    (property "Footprint" "Connector_PinHeader_1.00mm:PinHeader_1x02_P1.00mm_Vertical" (id 2) (at 67.564 178.308 0)
+      (effects (font (size 1.27 1.27)) hide)
+    )
+    (property "Datasheet" "~" (id 3) (at 67.564 178.308 0)
       (effects (font (size 1.27 1.27)) hide)
     )
@@
       (effects (font (size 1.524 1.524)))
     )
-    (property "Value" "" (id 1) (at 58.928 83.566 0)
+    (property "Value" "AMS1117-1.2" (id 1) (at 58.928 83.566 0)
       (effects (font (size 1.524 1.524)))
     )
@@
     (pin "1")
   )
+  (symbol (lib_id "jlcpcb-basic-mlcc-0402:100nF") (at 80.518 177.292 90) (unit 1)
+    (in_bom yes) (on_board yes)
+    (property "Reference" "C21" (id 0) (at 80.518 171.704 90))
+    (property "Value" "100nF" (id 1) (at 80.518 174.244 90))
+    (property "Footprint" "Capacitor_SMD:C_0402_1005Metric" (id 2) (at 84.328 176.3268 0)
+      (effects (font (size 1.27 1.27)) hide)
+    )
+    (property "Datasheet" "https://datasheet.lcsc.com/szlcsc/Samsung-Electro-Mechanics-CL05B104KO5NNNC_C1525.pdf" (id 3) (at 80.518 177.292 90)
+      (effects (font (size 1.27 1.27)) hide)
+    )
+    (property "LCSC" "C1525" (id 4) (at 80.518 177.292 90)
+      (effects (font (size 1.27 1.27)) hide)
+    )
+    (pin "1")
+    (pin "2")
+  )
   (sheet_instances
     (path "/" (page "1"))
@@
       (reference "C20") (unit 1) (value "100nF") (footprint "Capacitor_SMD:C_0805_2012Metric")
     )
+    (path "/fbf93733-a27a-4e7e-997f-2c561c90c6c2"
+      (reference "C21") (unit 1) (value "100nF") (footprint "Capacitor_SMD:C_0402_1005Metric")
+    )
+    (path "/6a3dd930-2f9e-49a7-b6e6-1af9239d0ebe"
+      (reference "C22") (unit 1) (value "100nF") (footprint "Capacitor_SMD:C_0402_1005Metric")
+    )
     (path "/0cafc14b-f536-4892-b5cc-930cd5178ba5"
