File: rev1/CH569Board.kicad_pcb (KiCad board)
At the start: 4 copper layers, 47.3 x 49.6 mm, 39 parts, among them CN1 BA42-80BT-1-NHB, J1 Conn_01x02_Male, J2 Conn_01x03_Male, U1 AMS1117-3.3, U2 AMS1117-1.2, U4 CH569W, X1 O705030MEEA4SC

Commit message: cosmetics
Routing:
- net +5V: track 55.1 -> 54.4 mm
- net GND: vias 83 -> 91
Changed lines of the file:
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@@
     (property "Sheetname" "")
     (attr smd)
-    (fp_text reference "C19" (at -0.02 -0.95) (layer "F.SilkS")
+    (fp_text reference "C19" (at -1.2 1.545 90) (layer "F.SilkS")
       (effects (font (size 0.5 0.5) (thickness 0.125)))
     )
@@
   )
   (segment (start 111.61 79.99) (end 111.61 84.79) (width 0.20574) (layer "F.Cu") (net 1))
-  (segment (start 114.81 84.79) (end 114.81 86.866) (width 0.20574) (layer "F.Cu") (net 1))
   (segment (start 118.81 84.79) (end 118.81 82.49) (width 0.20574) (layer "F.Cu") (net 1))
   (segment (start 130.81 82.44) (end 130.81 79.99) (width 0.20574) (layer "F.Cu") (net 1))
   (segment (start 114.81 84.79) (end 114.81 79.99) (width 0.20574) (layer "F.Cu") (net 1))
   (segment (start 129.8 114.230007) (end 129.8 115.92) (width 0.6) (layer "F.Cu") (net 1))
+  (segment (start 114.81 86.866) (end 114.81 84.79) (width 0.20574) (layer "F.Cu") (net 1))
   (segment (start 107.7976 87.9348) (end 108.964 87.9348) (width 0.20574) (layer "F.Cu") (net 1))
   (segment (start 102.23 118.071) (end 102.239 118.062) (width 1) (layer "F.Cu") (net 1))
@@
   (segment (start 139.12 121.992) (end 139.134 121.978) (width 1) (layer "F.Cu") (net 1))
   (segment (start 102.23 119.82) (end 102.23 118.071) (width 1) (layer "F.Cu") (net 1))
-  (segment (start 114.81 86.866) (end 114.808 86.868) (width 0.20574) (layer "F.Cu") (net 1))
   (segment (start 111.635 86.866) (end 111.633 86.868) (width 0.20574) (layer "F.Cu") (net 1))
   (segment (start 117.076887 104.57) (end 117.023147 104.51626) (width 1) (layer "F.Cu") (net 1))
@@
   (via (at 126.81 82.46) (size 0.45) (drill 0.2) (layers "F.Cu" "B.Cu") (net 1))
   (via (at 117.023147 104.51626) (size 0.95) (drill 0.8) (layers "F.Cu" "B.Cu") (net 1))
+  (via (at 114.525 98.175) (size 0.45) (drill 0.2) (layers "F.Cu" "B.Cu") (free) (net 1))
+  (via (at 113.5 100.125) (size 0.45) (drill 0.2) (layers "F.Cu" "B.Cu") (free) (net 1))
   (via (at 127.7112 105.521) (size 0.75) (drill 0.6) (layers "F.Cu" "B.Cu") (net 1))
+  (via (at 139.225 126.475) (size 0.45) (drill 0.2) (layers "F.Cu" "B.Cu") (free) (net 1))
   (via (at 118.17 119.51) (size 0.45) (drill 0.2) (layers "F.Cu" "B.Cu") (free) (net 1))
   (via (at 116.24 112.31) (size 0.45) (drill 0.2) (layers "F.Cu" "B.Cu") (free) (net 1))
   (via (at 127.7112 104.4542) (size 0.75) (drill 0.6) (layers "F.Cu" "B.Cu") (net 1))
-  (via (at 135.85 124.95) (size 0.45) (drill 0.2) (layers "F.Cu" "B.Cu") (free) (net 1))
+  (via (at 137.85 124.975) (size 0.45) (drill 0.2) (layers "F.Cu" "B.Cu") (free) (net 1))
+  (via (at 111.61 86.845) (size 0.45) (drill 0.2) (layers "F.Cu" "B.Cu") (net 1))
   (via (at 123.444 103.362) (size 0.75) (drill 0.6) (layers "F.Cu" "B.Cu") (net 1))
   (via (at 130.82 82.45) (size 0.45) (drill 0.2) (layers "F.Cu" "B.Cu") (net 1))
   (via (at 113.68 126.72) (size 0.45) (drill 0.2) (layers "F.Cu" "B.Cu") (free) (net 1))
   (via (at 109.54 82.52) (size 0.45) (drill 0.2) (layers "F.Cu" "B.Cu") (free) (net 1))
-  (via (at 102.58 122.56) (size 0.45) (drill 0.2) (layers "F.Cu" "B.Cu") (free) (net 1))
+  (via (at 106.85 123.6) (size 0.45) (drill 0.2) (layers "F.Cu" "B.Cu") (free) (net 1))
   (via (at 139.827 106.553) (size 0.45) (drill 0.2) (layers "F.Cu" "B.Cu") (free) (net 1))
   (via (at 118.79 109.75) (size 1.3) (drill 1) (layers "F.Cu" "B.Cu") (net 1))
@@
   (via (at 114.0714 106.6292) (size 0.45) (drill 0.2) (layers "F.Cu" "B.Cu") (free) (net 1))
   (via (at 124.5108 102.2952) (size 0.75) (drill 0.6) (layers "F.Cu" "B.Cu") (net 1))
+  (via (at 113.325 102.75) (size 0.45) (drill 0.2) (layers "F.Cu" "B.Cu") (free) (net 1))
   (via (at 117.62 110.66) (size 0.45) (drill 0.2) (layers "F.Cu" "B.Cu") (free) (net 1))
   (via (at 126.6444 102.3206) (size 0.75) (drill 0.6) (layers "F.Cu" "B.Cu") (net 1))
@@
   (via (at 123.444 104.4288) (size 0.75) (drill 0.6) (layers "F.Cu" "B.Cu") (net 1))
   (via (at 142.99 94.17) (size 0.45) (drill 0.2) (layers "F.Cu" "B.Cu") (free) (net 1))
+  (via (at 111.125 92.575) (size 0.45) (drill 0.2) (layers "F.Cu" "B.Cu") (free) (net 1))
   (via (at 141.986 97.663) (size 0.45) (drill 0.2) (layers "F.Cu" "B.Cu") (free) (net 1))
   (via (at 123.444 105.4956) (size 0.75) (drill 0.6) (layers "F.Cu" "B.Cu") (net 1))
@@
   (via (at 138.81 82.39) (size 0.45) (drill 0.2) (layers "F.Cu" "B.Cu") (net 1))
   (via (at 101.37 120.69) (size 0.45) (drill 0.2) (layers "F.Cu" "B.Cu") (free) (net 1))
+  (via (at 145.65 126.45) (size 0.45) (drill 0.2) (layers "F.Cu" "B.Cu") (free) (net 1))
   (via (at 124.5108 101.203) (size 0.75) (drill 0.6) (layers "F.Cu" "B.Cu") (net 1))
   (via (at 129.84 119.47) (size 0.45) (drill 0.2) (layers "F.Cu" "B.Cu") (free) (net 1))
@@
   (via (at 117.3988 109.6772) (size 0.45) (drill 0.2) (layers "F.Cu" "B.Cu") (free) (net 1))
   (via (at 121.08 98.06) (size 0.45) (drill 0.2) (layers "F.Cu" "B.Cu") (free) (net 1))
+  (via (at 114.5 96.075) (size 0.45) (drill 0.2) (layers "F.Cu" "B.Cu") (free) (net 1))
   (via (at 134.81 82.38) (size 0.45) (drill 0.2) (layers "F.Cu" "B.Cu") (net 1))
   (via (at 141.986 104.394) (size 0.45) (drill 0.2) (layers "F.Cu" "B.Cu") (free) (net 1))
@@
   (segment (start 108.528 118.062) (end 114.0624 123.5964) (width 1) (layer "In2.Cu") (net 3))
   (segment (start 114.0624 123.5964) (end 144.5768 123.5964) (width 1) (layer "In2.Cu") (net 3))
-  (segment (start 108.528 118.062) (end 108.528 118.788) (width 1) (layer "In2.Cu") (net 3))
   (segment (start 145.8968 122.2764) (end 145.8968 121.958) (width 1) (layer "In2.Cu") (net 3))
   (segment (start 144.5768 123.5964) (end 145.8968 122.2764) (width 1) (layer "In2.Cu") (net 3))
@@
   (segment (start 113.298347 83.885147) (end 115.395493 81.788) (width 0.2) (layer "B.Cu") (net 32))
   (segment (start 116.205 81.788) (end 116.459 81.534) (width 0.2) (layer "B.Cu") (net 32))
-  (segment (start 113.109493 84.074) (end 113.298347 83.885147) (width 0.2) (layer "B.Cu") (net 32))
   (segment (start 116.586 96.52) (end 112.268 92.202) (width 0.2) (layer "B.Cu") (net 32))
   (segment (start 112.268 84.915494) (end 113.298347 83.885147) (width 0.2) (layer "B.Cu") (net 32))

Commit message: fix important flaw in rev1: 3.3V and VIO were not connected
Parts:
- removed N1: OHWLOGO, Symbols:OSHW-Symbol_6.7x6mm_SilkScreen
Connections:
- C15 pad 1: /VIO -> +3V3
- C8 pad 1: /VIO -> +3V3
- U4 pad 16: /VIO -> +3V3
- U4 pad 42: /VIO -> +3V3
- U4 pad 61: /VIO -> +3V3
Routing:
- net +3V3: track 65.8 -> 91.9 mm, vias 4 -> 7
- net /VIO: track 25.1 -> 0.00 mm, vias 3 -> 0
