File: rev1/CH569Board.kicad_sch (KiCad schematic)
At the start: 38 parts, among them CN1 BA42-80BT-1-NHB, J1 Conn_01x02_Male, J2 Conn_01x03_Male, U1 AMS1117-3.3, U2 AMS1117-1.2, U4 CH569W, X1 O705030MEEA4SC

Commit message: cosmetics
Other:
- moved on the sheet: C21, C22, J1
Changed lines of the file:
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@@
+    (stroke (width 0) (type default) (color 0 0 0 0))
+  )
+  (wire (pts (xy 133.096 59.436) (xy 156.21 59.436))
     (stroke (width 0) (type default) (color 0 0 0 0))
   )
@@
     (stroke (width 0) (type default) (color 0 0 0 0))
   )
+  (wire (pts (xy 76.962 169.418) (xy 76.962 170.434))
+    (stroke (width 0) (type default) (color 0 0 0 0))
+  )
   (wire (pts (xy 157.48 129.286) (xy 150.114 129.286))
     (stroke (width 0) (type default) (color 0 0 0 0))
@@
     (stroke (width 0) (type default) (color 0 0 0 0))
   )
-  (wire (pts (xy 77.978 177.292) (xy 72.644 177.292))
+  (wire (pts (xy 76.962 166.116) (xy 87.376 166.116))
     (stroke (width 0) (type default) (color 0 0 0 0))
   )
@@
     (stroke (width 0) (type default) (color 0 0 0 0))
   )
+  (wire (pts (xy 76.962 166.116) (xy 76.962 166.878))
+    (stroke (width 0) (type default) (color 0 0 0 0))
+  )
   (wire (pts (xy 248.92 91.948) (xy 256.032 91.948))
     (stroke (width 0) (type default) (color 0 0 0 0))
@@
     (stroke (width 0) (type default) (color 0 0 0 0))
   )
-  (wire (pts (xy 90.17 181.61) (xy 83.058 181.61))
+  (wire (pts (xy 99.568 170.434) (xy 92.456 170.434))
     (stroke (width 0) (type default) (color 0 0 0 0))
   )
@@
     (stroke (width 0) (type default) (color 0 0 0 0))
   )
+  (wire (pts (xy 149.098 54.356) (xy 156.21 54.356))
+    (stroke (width 0) (type default) (color 0 0 0 0))
+  )
   (wire (pts (xy 51.816 155.448) (xy 44.704 155.448))
     (stroke (width 0) (type default) (color 0 0 0 0))
@@
     (stroke (width 0) (type default) (color 0 0 0 0))
   )
-  (wire (pts (xy 90.17 177.292) (xy 83.058 177.292))
+  (wire (pts (xy 99.568 166.116) (xy 92.456 166.116))
     (stroke (width 0) (type default) (color 0 0 0 0))
   )
@@
     (stroke (width 0) (type default) (color 0 0 0 0))
   )
-  (wire (pts (xy 133.096 59.436) (xy 156.21 59.436))
-    (stroke (width 0) (type default) (color 0 0 0 0))
-  )
   (wire (pts (xy 161.798 157.226) (xy 168.402 157.226))
     (stroke (width 0) (type default) (color 0 0 0 0))
@@
     (stroke (width 0) (type default) (color 0 0 0 0))
   )
-  (wire (pts (xy 72.644 177.292) (xy 72.644 178.308))
-    (stroke (width 0) (type default) (color 0 0 0 0))
-  )
   (wire (pts (xy 166.624 99.314) (xy 171.196 99.314))
     (stroke (width 0) (type default) (color 0 0 0 0))
@@
     (stroke (width 0) (type default) (color 0 0 0 0))
   )
-  (wire (pts (xy 72.644 181.61) (xy 72.644 180.848))
-    (stroke (width 0) (type default) (color 0 0 0 0))
-  )
   (wire (pts (xy 120.65 64.77) (xy 133.096 64.77))
     (stroke (width 0) (type default) (color 0 0 0 0))
@@
     (stroke (width 0) (type default) (color 0 0 0 0))
   )
-  (wire (pts (xy 77.978 181.61) (xy 72.644 181.61))
+  (wire (pts (xy 76.962 170.434) (xy 87.376 170.434))
     (stroke (width 0) (type default) (color 0 0 0 0))
   )
@@
   )
   (wire (pts (xy 157.226 116.586) (xy 150.114 116.586))
-    (stroke (width 0) (type default) (color 0 0 0 0))
-  )
-  (wire (pts (xy 149.098 54.356) (xy 156.21 54.356))
     (stroke (width 0) (type default) (color 0 0 0 0))
   )
@@
     (effects (font (size 1.27 1.27)) (justify left bottom))
   )
-  (label "GX+" (at 85.344 177.292 0)
+  (label "GX+" (at 94.742 166.116 0)
     (effects (font (size 1.27 1.27)) (justify left bottom))
   )
@@
     (effects (font (size 1.27 1.27)) (justify left bottom))
   )
-  (label "GXO-" (at 73.66 181.61 0)
+  (label "GXO-" (at 83.058 170.434 0)
     (effects (font (size 1.27 1.27)) (justify left bottom))
   )
@@
     (effects (font (size 1.27 1.27)) (justify left bottom))
   )
-  (label "GX-" (at 85.344 181.61 0)
+  (label "GX-" (at 94.742 170.434 0)
     (effects (font (size 1.27 1.27)) (justify left bottom))
   )
@@
     (effects (font (size 1.27 1.27)) (justify right bottom))
   )
-  (label "GXO+" (at 73.66 177.292 0)
+  (label "GXO+" (at 83.058 166.116 0)
     (effects (font (size 1.27 1.27)) (justify left bottom))
   )
@@
     (pin "1")
   )
-  (symbol (lib_id "jlcpcb-basic-mlcc-0402:100nF") (at 80.518 181.61 90) (unit 1)
-    (in_bom yes) (on_board yes)
-    (property "Reference" "C22" (id 0) (at 80.518 185.166 90))
-    (property "Value" "100nF" (id 1) (at 80.518 187.706 90))
-    (property "Footprint" "Capacitor_SMD:C_0402_1005Metric" (id 2) (at 84.328 180.6448 0)
-      (effects (font (size 1.27 1.27)) hide)
-    )
-    (property "Datasheet" "https://datasheet.lcsc.com/szlcsc/Samsung-Electro-Mechanics-CL05B104KO5NNNC_C1525.pdf" (id 3) (at 80.518 181.61 90)
-      (effects (font (size 1.27 1.27)) hide)
-    )
-    (property "LCSC" "C1525" (id 4) (at 80.518 181.61 90)
+  (symbol (lib_id "jlcpcb-basic-mlcc-0402:100nF") (at 89.916 170.434 90) (unit 1)
+    (in_bom yes) (on_board yes)
+    (property "Reference" "C22" (id 0) (at 89.916 173.99 90))
+    (property "Value" "100nF" (id 1) (at 89.916 176.53 90))
+    (property "Footprint" "Capacitor_SMD:C_0402_1005Metric" (id 2) (at 93.726 169.4688 0)
+      (effects (font (size 1.27 1.27)) hide)
+    )
+    (property "Datasheet" "https://datasheet.lcsc.com/szlcsc/Samsung-Electro-Mechanics-CL05B104KO5NNNC_C1525.pdf" (id 3) (at 89.916 170.434 90)
+      (effects (font (size 1.27 1.27)) hide)
+    )
+    (property "LCSC" "C1525" (id 4) (at 89.916 170.434 90)
       (effects (font (size 1.27 1.27)) hide)
     )
@@
       (effects (font (size 1.27 1.27)) hide)
     )
-    (property "Value" "GND" (id 1) (at 133.477 81.7118 0))
+    (property "Value" "GND" (id 1) (at 129.54 84.582 0))
     (property "Footprint" "" (id 2) (at 133.604 86.106 0)
       (effects (font (size 1.27 1.27)) hide)
@@
     (pin "1")
   )
-  (symbol (lib_id "Connector:Conn_01x02_Male") (at 67.564 178.308 0) (unit 1)
-    (in_bom yes) (on_board yes)
-    (property "Reference" "J1" (id 0) (at 67.564 176.276 0))
-    (property "Value" "Conn_01x02_Male" (id 1) (at 72.39 183.388 0))
-    (property "Footprint" "Connector_PinHeader_2.54mm:PinHeader_1x02_P2.54mm_Vertical" (id 2) (at 67.564 178.308 0)
-      (effects (font (size 1.27 1.27)) hide)
-    )
-    (property "Datasheet" "~" (id 3) (at 67.564 178.308 0)
+  (symbol (lib_id "Connector:Conn_01x02_Male") (at 71.882 166.878 0) (unit 1)
+    (in_bom yes) (on_board yes)
+    (property "Reference" "J1" (id 0) (at 71.882 164.846 0))
+    (property "Value" "Conn_01x02_Male" (id 1) (at 76.708 171.958 0)
+      (effects (font (size 1.27 1.27)) hide)
+    )
+    (property "Footprint" "Connector_PinHeader_2.54mm:PinHeader_1x02_P2.54mm_Vertical" (id 2) (at 71.882 166.878 0)
+      (effects (font (size 1.27 1.27)) hide)
+    )
+    (property "Datasheet" "~" (id 3) (at 71.882 166.878 0)
       (effects (font (size 1.27 1.27)) hide)
     )
@@
     (pin "1")
   )
-  (symbol (lib_id "jlcpcb-basic-mlcc-0402:100nF") (at 80.518 177.292 90) (unit 1)
-    (in_bom yes) (on_board yes)
-    (property "Reference" "C21" (id 0) (at 80.518 171.704 90))
-    (property "Value" "100nF" (id 1) (at 80.518 174.244 90))
-    (property "Footprint" "Capacitor_SMD:C_0402_1005Metric" (id 2) (at 84.328 176.3268 0)
-      (effects (font (size 1.27 1.27)) hide)
-    )
-    (property "Datasheet" "https://datasheet.lcsc.com/szlcsc/Samsung-Electro-Mechanics-CL05B104KO5NNNC_C1525.pdf" (id 3) (at 80.518 177.292 90)
-      (effects (font (size 1.27 1.27)) hide)
-    )
-    (property "LCSC" "C1525" (id 4) (at 80.518 177.292 90)
-      (effects (font (size 1.27 1.27)) hide)
-    )
+  (symbol (lib_id "jlcpcb-basic-mlcc-0402:100nF") (at 89.916 166.116 90) (unit 1)
+    (in_bom yes) (on_board yes)
+    (property "Reference" "C21" (id 0) (at 89.916 160.528 90))
+    (property "Value" "100nF" (id 1) (at 89.916 163.068 90))
+    (property "Footprint" "Capacitor_SMD:C_0402_1005Metric" (id 2) (at 93.726 165.1508 0)
+      (effects (font (size 1.27 1.27)) hide)
+    )
+    (property "Datasheet" "https://datasheet.lcsc.com/szlcsc/Samsung-Electro-Mechanics-CL05B104KO5NNNC_C1525.pdf" (id 3) (at 89.916 166.116 90)
+      (effects (font (size 1.27 1.27)) hide)
+    )
+    (property "LCSC" "C1525" (id 4) (at 89.916 166.116 90)
+      (effects (font (size 1.27 1.27)) hide)
+    )

Commit message: fix important flaw in rev1: 3.3V and VIO were not connected
Connections:
- net VIO is gone; now on net +3V3: C15.1, C8.1, U4.16 (VDDIO), U4.42 (VDDIO), U4.61 (VDDIO)
Changed lines of the file:
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@@
+    (stroke (width 0) (type default) (color 0 0 0 0))
+  )
+  (wire (pts (xy 90.424 129.286) (xy 90.424 127.762))
     (stroke (width 0) (type default) (color 0 0 0 0))
   )
@@
     (stroke (width 0) (type default) (color 0 0 0 0))
   )
-  (wire (pts (xy 92.964 129.286) (xy 96.774 129.286))
+  (wire (pts (xy 90.424 129.286) (xy 96.774 129.286))
     (stroke (width 0) (type default) (color 0 0 0 0))
   )
@@
     (pin "9")
   )
+  (symbol (lib_id "power:+3V3") (at 90.424 127.762 0) (mirror y) (unit 1)
+    (in_bom yes) (on_board yes) (fields_autoplaced)
+    (property "Reference" "#PWR?" (id 0) (at 90.424 131.572 0)
+      (effects (font (size 1.27 1.27)) hide)
+    )
+    (property "Value" "+3V3" (id 1) (at 92.71 126.4919 0)
+      (effects (font (size 1.27 1.27)) (justify right))
+    )
+    (property "Footprint" "" (id 2) (at 90.424 127.762 0)
+      (effects (font (size 1.27 1.27)) hide)
+    )
+    (property "Datasheet" "" (id 3) (at 90.424 127.762 0)
+      (effects (font (size 1.27 1.27)) hide)
+    )
+    (pin "1")
+  )
   (symbol (lib_id "power:GND") (at 96.774 134.366 0) (unit 1)
     (in_bom yes) (on_board yes)
@@
       (reference "#PWR059") (unit 1) (value "GND") (footprint "")
     )
+    (path "/0cdee745-671e-4f02-894c-e7317ebcd74b"
+      (reference "#PWR?") (unit 1) (value "+3V3") (footprint "")
+    )
     (path "/24a026b0-25b7-4804-8e60-d3054b977236"
