File: rev2/CH569Board.kicad_sch (KiCad schematic)
At the start: 35 parts, among them CN1 BA42-80BT-1-NHB, J1 Conn_01x02_Male, J2 Conn_01x03_Male, U1 AMS1117-3.3, U4 CH569W, X1 O705030MEEA4SC

Commit message: redo power section with different LDO, add decoupling cap and reset switch
Parts:
- removed U1: AMS1117-3.3, easyeda2kicad:SOT-223-3_L6.5-W3.4-P2.30-LS7.0-BR, symbol easyeda2kicad:AMS1117-3.3
- added C2, C3: 1uF, C_0805_2012Metric, symbol jlcpcb-basic-mlcc-0805:1uF
- added C5: 100nF, Capacitor_SMD:C_0402_1005Metric, symbol jlcpcb-basic-mlcc-0402:100nF
- added R6: 10k, R_0402_1005Metric, symbol jlcpcb-basic-resistor-0402:10k
- added SW1: TS-1187A-B-A-B, SW-SMD_4P-L5.1-W5.1-P3.70-LS6.5-TL-2, symbol easyeda2kicad:TS-1187A-B-A-B
- added U1: SPX3819M5-L-3-3/TR, easyeda2kicad:SOT-23-5_L3.0-W1.7-P0.95-LS2.8-BR, symbol easyeda2kicad:SPX3819M5-L-3-3/TR
Connections:
- net +3V3: now also C2.1, C5.1, U1.5 (OUT)
- net +5V: now also R6.2, U1.1 (IN)
- net GND: now also C2.2, C3.2, C5.2, SW1.3 (C), SW1.4 (D), U1.2 (GND)
- new net: C3.1, U1.4 (BYP)
- new net: R6.1, SW1.1 (A), SW1.2 (B), U1.3 (EN)
Other:
- moved on the sheet: C1

Commit message: rev2 ready for the fab. used a crystal instead of an XO, because of better specs
Parts:
- removed C5: 100nF, Capacitor_SMD:C_0402_1005Metric, symbol jlcpcb-basic-mlcc-0402:100nF
- removed R1: 10k, Resistor_SMD:R_0603_1608Metric, symbol Device:R_Small
- removed X1: O705030MEEA4SC, easyeda2kicad:OSC-SMD_4P-L7.0-W5.0-BL, symbol easyeda2kicad:O705030MEEA4SC
- added C23, C5: 10pF, C_0402_1005Metric, symbol jlcpcb-basic-mlcc-0402:10pF
- added X1: X1E0000210295, CRYSTAL-SMD_4P-L3.2-W2.5-BL, symbol easyeda2kicad:X1E0000210295
Connections:
- net GND: now also C23.2, C5.2, X1.2 (GND), X1.4 (GND)
- net XI: now also C5.1, X1.1 (OSC1)
- net XO: now reaches U4.67 (XO)
- net XO: now also C23.1, X1.3 (OSC2)
- no-connect marks 20 -> 19
